Commit message: removed unnecessary axes from the chain urdf

File: examples/rsc/chain/robot.urdf (robot description, URDF)
Before this commit: robot 2DrobotArm, 5 links, 4 joints
Joints:
- joint link1Tolink2: axis 0 1 0 -> (none)
- joint link2Tolink3: axis 0 1 0 -> (none)
- joint link3Tolink4: axis 0 1 0 -> (none)

Commit message: kinova example now had many arms. background in newtonsCradle example. chain urdf removed unncessary axis param

File: examples/rsc/chain/robot.urdf (robot description, URDF)
Before this commit: robot 2DrobotArm, 5 links, 4 joints
Joints:
- joint link3Tolink4: limit lower=1 -> (none)

Commit message: complated compound but need testing

File: examples/rsc/chain/robot.urdf (robot description, URDF)
Before this commit: robot 2DrobotArm, 5 links, 4 joints
Joints:
- joint link1Tolink2: limit lower=1 -> lower=1.5
